File: PCB/PiicoDev-Precision-Temperature-Sensor-TMP117.kicad_sch (KiCad schematic)
At the start: 24 parts, among them J1 , J2 , J3 , SW1 SW_DIP_x04, U1 TMP117

Commit message: add v12 comments, update schematic pdf
Other:
- note added: "ASW: Only one switch to be ON at a time 1 2 3 4 I2C Address [ON OFF OFF OFF] 0x48 [OFF ON OFF OFF] 0x49 [OFF OFF ON OFF] 0x4A [OFF OFF OFF ON ] 0x4B If no ASW set, address appears to default to 0x48"
- note removed: "ASW 1 2 3 4 [ON OFF OFF OFF] 0x48 [OFF ON OFF OFF] 0x49 [OFF OFF ON OFF] 0x4A [OFF OFF OFF ON ] 0x4B"
Changed lines of the file:
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@@
     (effects (font (size 1.27 1.27)) (justify left bottom))
   )
-  (text "ASW\n  1    2   3   4\n[ON  OFF OFF OFF] 0x48\n[OFF ON  OFF OFF] 0x49\n[OFF OFF ON  OFF] 0x4A\n[OFF OFF OFF ON ] 0x4B"
+  (text "ASW: Only one switch to be ON at a time\n\n  1    2   3   4      I2C Address\n[ON  OFF OFF OFF]     0x48\n[OFF ON  OFF OFF]     0x49\n[OFF OFF ON  OFF]     0x4A\n[OFF OFF OFF ON ]     0x4B\n\nIf no ASW set, address appears to default to 0x48"
     (at 139.7 123.19 0)
     (effects (font (size 1.27 1.27)) (justify left bottom))
